File: SoundProcessorV2.kicad_pcb (KiCad board)
At the start: 2 copper layers, 100 x 60 mm, 44 parts, among them P1 CONN_01X04, P2 CONN_01X04, P3 CONN_01X03, P4 CONN_01X05, P5 CONN_01X05, U1 TDA1524, U2 AD5206, U3 MSGEQ7, U4 MSGEQ7

Commit message: Poprawiono zasilanie i wejscie do wizualizera
Parts:
- removed the REF** at (110.4, 56.6)
- P4, P5: footprint Pin_Headers:Pin_Header_Straight_1x04 -> Pin_Headers:Pin_Header_Straight_1x05
Connections:
- P4 pad 2: Net-(P4-Pad2) -> Net-(C2-Pad2)
- P5 pad 2: Net-(P5-Pad2) -> Net-(C1-Pad2)
- R8 pad 2: Net-(P4-Pad2) -> Net-(C2-Pad2)
- R9 pad 2: Net-(P5-Pad2) -> Net-(R9-Pad2)
Routing:
- net +5V: track 95.8 -> 148.3 mm
- net Net-(C2-Pad2): track 8.49 -> 48.6 mm
- net Net-(C1-Pad2): track 7.34 -> 24.8 mm
- net Net-(P4-Pad5): track 0.00 -> 12.9 mm
- net Net-(P5-Pad5): track 0.00 -> 12.4 mm
- net Net-(P5-Pad2): track 11.2 -> 0.00 mm
- net Net-(P4-Pad2): track 10.4 -> 0.00 mm
- net Net-(R9-Pad2): track 0.00 -> 1.91 mm
