File: V3/Zasilacz.kicad_pcb (KiCad board)
At the start: 2 copper layers, 32 parts, among them J1 CONN_01X02, J2 CONN_01X04, J3 CONN_01X04, J4 CONN_01X02, U1 LM317_SOT223, U2 LM317_SOT223

Commit message: Zasilacz v1
Routing:
- net Net-(C1-Pad1): track 55.0 -> 7.30 mm
- net Net-(C7-Pad1): track 50.6 -> 5.66 mm
- net Earth: track 179.2 -> 167.8 mm
Other:
- board text added: "+"
- board text added: "-"
Changed lines of the file:
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@@
     (links 58)
     (no_connects 1)
-    (area 0 0 0 0)
+    (area 27.828 119.974999 141.55 196.100001)
     (thickness 1.6)
-    (drawings 9)
-    (tracks 123)
+    (drawings 11)
+    (tracks 100)
     (zones 0)
     (modules 32)
@@
   )
   (setup
-    (last_trace_width 1)
+    (last_trace_width 0.25)
     (user_trace_width 0.5)
     (user_trace_width 0.75)
@@
     (visible_elements FFFFFF7F)
     (pcbplotparams
-      (layerselection 0x00030_80000001)
+      (layerselection 0x00000_00000001)
       (usegerberextensions false)
       (excludeedgelayer true)
@@
       (padsonsilk false)
       (subtractmaskfromsilk false)
-      (outputformat 1)
+      (outputformat 4)
       (mirror false)
       (drillshape 1)
@@
     (pad 1 thru_hole circle (at 0 0) (size 4.064 4.064) (drill 3.048) (layers *.Cu *.Mask F.SilkS))
   )
+  (gr_text - (at 31.1 158.45 90) (layer F.Cu)
+    (effects (font (size 1.5 1.5) (thickness 0.3)))
+  )
+  (gr_text + (at 31.35 153.4) (layer F.Cu)
+    (effects (font (size 1.5 1.5) (thickness 0.3)))
+  )
   (target plus (at 49.95 156.1) (size 5) (width 0.15) (layer Edge.Cuts))
   (target plus (at 124.7 187.85) (size 5) (width 0.15) (layer Edge.Cuts))
@@
   (segment (start 61.10254 140.60052) (end 61.10254 133.80254) (width 1) (layer F.Cu) (net 1))
   (segment (start 61.10254 133.80254) (end 60.75 133.45) (width 1) (layer F.Cu) (net 1))
-  (segment (start 61.10254 140.60052) (end 57.28948 140.60052) (width 1) (layer F.Cu) (net 1))
-  (segment (start 57.28948 140.60052) (end 56.14 141.75) (width 1) (layer F.Cu) (net 1))
-  (segment (start 61.10254 140.60052) (end 78.40052 140.60052) (width 1) (layer F.Cu) (net 1))
-  (segment (start 78.40052 140.60052) (end 80.8 143) (width 1) (layer F.Cu) (net 1))
-  (segment (start 102.4 143) (end 80.8 143) (width 1) (layer F.Cu) (net 1))
   (segment (start 47.15 189.06) (end 34.06 189.06) (width 1) (layer F.Cu) (net 2))
   (segment (start 32.55 187.55) (end 32.55 177.6) (width 1) (layer F.Cu) (net 2))
@@
   (segment (start 50.75 123.45) (end 44.25 123.45) (width 1) (layer F.Cu) (net 2))
   (segment (start 44.25 123.45) (end 35.2 123.45) (width 1) (layer F.Cu) (net 2))
-  (segment (start 32.7 144.6) (end 36.55 148.45) (width 1) (layer F.Cu) (net 2))
-  (segment (start 32.7 140.45) (end 32.7 144.6) (width 1) (layer F.Cu) (net 2))
-  (segment (start 34 139.15) (end 32.7 140.45) (width 1) (layer F.Cu) (net 2))
   (segment (start 34 124.65) (end 34 125.45) (width 1) (layer F.Cu) (net 2))
   (segment (start 34 125.45) (end 34 137.6) (width 1) (layer F.Cu) (net 2))
@@
   (segment (start 47.80052 173.14746) (end 50.5 175.84694) (width 1) (layer F.Cu) (net 5))
   (segment (start 50.5 175.84694) (end 50.5 178.9) (width 1) (layer F.Cu) (net 5))
-  (segment (start 53.6 141.75) (end 53.6 144.8) (width 1.5) (layer F.Cu) (net 6))
-  (segment (start 45.2 136.76) (end 45.2 134.85) (width 1) (layer F.Cu) (net 6))
-  (segment (start 43.95 133.6) (end 37.8 133.6) (width 1) (layer F.Cu) (net 6))
-  (segment (start 45.2 134.85) (end 43.95 133.6) (width 1) (layer F.Cu) (net 6))
-  (segment (start 42 141.15) (end 42 138.2) (width 1) (layer F.Cu) (net 6))
-  (segment (start 42 138.2) (end 42 137.8) (width 1) (layer F.Cu) (net 6))
-  (segment (start 42 137.8) (end 37.8 133.6) (width 1) (layer F.Cu) (net 6))
-  (segment (start 36.55 153.45) (end 38.05 153.45) (width 1) (layer F.Cu) (net 6))
-  (segment (start 38.05 153.45) (end 42 149.5) (width 1) (layer F.Cu) (net 6))
-  (segment (start 42 149.5) (end 42 141.15) (width 1) (layer F.Cu) (net 6))
-  (segment (start 55.65 147.7) (end 54.85 147.7) (width 1) (layer F.Cu) (net 6))
-  (segment (start 54.85 147.7) (end 53.6 146.45) (width 1) (layer F.Cu) (net 6))
-  (segment (start 53.6 146.45) (end 53.6 144.8) (width 1) (layer F.Cu) (net 6))
-  (segment (start 55.44948 150.75254) (end 55.44948 147.90052) (width 1) (layer F.Cu) (net 6))
-  (segment (start 55.44948 147.90052) (end 55.65 147.7) (width 1) (layer F.Cu) (net 6))
-  (segment (start 61.10254 150.76052) (end 55.45746 150.76052) (width 1) (layer F.Cu) (net 6))
-  (segment (start 55.45746 150.76052) (end 55.44948 150.75254) (width 1) (layer F.Cu) (net 6))
+  (segment (start 55.44948 150.75254) (end 61.09456 150.75254) (width 1) (layer F.Cu) (net 6))
+  (segment (start 61.09456 150.75254) (end 61.10254 150.76052) (width 1) (layer F.Cu) (net 6))
   (segment (start 36.35 177.6) (end 36.35 176.6) (width 1) (layer F.Cu) (net 7))
   (segment (start 37.5 175.45) (end 42.3 175.45) (width 1) (layer F.Cu) (net 7))
@@
     (polygon
       (pts
-        (xy 105.2 149.6) (xy 98.8 149.6) (xy 98.95 155.15) (xy 59.45 155.15) (xy 59.45 144.85)
-        (xy 55.15 144.9) (xy 55.15 139.95) (xy 62.65 140) (xy 62.65 138.9) (xy 93.45 138.7)
-        (xy 105.35 138.7)
+        (xy 105.4 149.6) (xy 98.8 149.6) (xy 98.8 155.15) (xy 59.45 155.15) (xy 59.45 144.85)
+        (xy 55.15 144.85) (xy 55.15 140) (xy 62.65 140) (xy 62.65 138.7) (xy 93.45 138.7)
+        (xy 105.4 138.7)
       )
     )
@@
     (polygon
       (pts
-        (xy 58.3 155.5) (xy 32.3 155.55) (xy 32.15 151.45) (xy 38.85 151.4) (xy 39.05 141.45)
-        (xy 37.55 141.45) (xy 37.3 131.6) (xy 48.8 131.45) (xy 48.75 143.25) (xy 52.05 143.25)
-        (xy 52.05 140.05) (xy 54.55 140.05) (xy 54.55 145.45) (xy 58.4 145.45) (xy 58.4 155.1)
+        (xy 58.4 155.5) (xy 32.3 155.55) (xy 32.3 151.45) (xy 39.05 151.45) (xy 39.05 144.5)
+        (xy 36.7 144.5) (xy 36.7 131.65) (xy 48.8 131.55) (xy 48.85 143.3) (xy 52.05 143.25)
+        (xy 52.05 140.05) (xy 54.6 140.05) (xy 54.6 145.45) (xy 58.4 145.45) (xy 58.4 155.1)
       )
     )
@@
     (polygon
       (pts
-        (xy 107.95 134.35) (xy 115.5 134.35) (xy 115.4 145) (xy 127.4 145) (xy 127.75 165.9)
-        (xy 127.75 166.55) (xy 116.35 166.65) (xy 116.35 178.8) (xy 108.1 178.7) (xy 108.1 191.35)
+        (xy 107.95 134.45) (xy 115.4 134.45) (xy 115.4 145) (xy 129.75 145) (xy 129.65 166.55)
+        (xy 127.75 166.55) (xy 116.35 166.65) (xy 116.4 178.7) (xy 108.1 178.7) (xy 108.1 191.35)
         (xy 29.95 191.35) (xy 30.05 161.5) (xy 31.386758 161.3) (xy 39.8 161.3) (xy 39.8 177.1)
         (xy 59.65 177.1) (xy 59.65 175.6) (xy 107.3 175.6) (xy 107.3 164) (xy 114.35 164)
         (xy 114.35 149.45) (xy 107.2 149.45) (xy 107.2 138.4) (xy 105.85 137.05) (xy 59.5 137.05)
-        (xy 59.5 139.1) (xy 52.1 139.1) (xy 52.1 130.5) (xy 35.35 130.5) (xy 35.35 145.85)
+        (xy 59.5 139.1) (xy 52.1 139.1) (xy 52.1 130.5) (xy 35.6 130.55) (xy 35.6 145.9)
         (xy 36.9 145.85) (xy 36.9 150.45) (xy 31.3 150.45) (xy 31.3 150.55) (xy 30 150.45)
-        (xy 30 121.45) (xy 108.2 121.45)
+        (xy 30 121.45) (xy 107.95 121.45)
       )
     )
@@
     (polygon
       (pts
-        (xy 127.75 143.5) (xy 127.75 128.1) (xy 109.1 128.1) (xy 109.1 133.6) (xy 120.35 133.6)
+        (xy 129.7 143.5) (xy 129.7 128.1) (xy 109.1 128.1) (xy 109.1 133.6) (xy 120.35 133.6)
         (xy 120.35 143.5) (xy 127.7 143.5) (xy 127.7 143.45)
       )
@@
     (polygon
       (pts
-        (xy 113.4 156) (xy 100.35 156) (xy 100.35 151.5) (xy 100.35 150.2) (xy 113.35 150.3)
+        (xy 113.4 156) (xy 100.35 156) (xy 100.35 151.5) (xy 100.35 150.3) (xy 113.4 150.3)
       )
     )
@@
     (polygon
       (pts
-        (xy 127.8 185.4) (xy 109.1 185.4) (xy 109.1 179.65) (xy 120.2 179.65) (xy 120.2 169.4)
-        (xy 127.8 169.4)
+        (xy 129.575 185.375) (xy 109.1 185.4) (xy 109.1 179.65) (xy 120.2 179.65) (xy 120.2 169.4)
+        (xy 129.575 169.375)
       )
     )
@@
       )
     )
-  )
-  (zone (net 3) (net_name "Net-(C2-Pad2)") (layer F.Cu) (hatch edge 0.508)
-    (connect_pads (clearance 0.508))
-    (min_thickness 0.254)
-    (fill yes (arc_segments 16) (thermal_gap 0.508) (thermal_bridge_width 0.508))
-    (polygon
-      (pts
-        (xy 105.3 164.2) (xy 105.45 164.2) (xy 105.45 164.25) (xy 105.3 164.25)
-      )
-    )

Commit message: Zasilcz poprawkiw sciezkach
Parts:
- moved D3 101.7 mm to (60.6, 65.8)
- moved R4 101.7 mm to (57.9, 65.8)
- moved C1 101.7 mm to (81.0, 41.3)
- moved C4 101.7 mm to (60.8, 72.2)
- moved C5 101.7 mm to (55.4, 27.2)
- moved C6 101.7 mm to (55.2, 79.3)
- moved C9 101.7 mm to (42.1, 39.5)
- moved D1 101.7 mm to (102.5, 52.2)
- moved D4 101.7 mm to (55.6, 49.0)
- moved D5 101.7 mm to (47.8, 69.0)
- moved D6 101.7 mm to (39.2, 25.1)
- moved J1 101.7 mm to (123.5, 74.8)
- moved J3 101.7 mm to (123.5, 62.3)
- moved J4 101.7 mm to (123.5, 39.8)
- moved R2 101.7 mm to (50.6, 77.2)
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Routing:
- net Earth: track 167.8 -> 29.8 mm
- net Net-(C2-Pad2): track 81.6 -> 0.65 mm
- net AC: track 41.1 -> 10.0 mm
- net Net-(C10-Pad1): track 37.8 -> 13.8 mm
- net Net-(D1-Pad3): track 9.04 -> 0.14 mm
- net Net-(D1-Pad2): track 8.94 -> 0.14 mm
