File: V3/SoftStart/SoftStart.kicad_pcb (KiCad board)
At the start: 2 copper layers, 32 parts, among them J1 CONN_01X04, J3 CONN_01X01, J4 CONN_01X04, J5 CONN_01X04, J6 CONN_02X03, Q1 Q_NPN_BCE, T1 Transformer_1P_2S, U1 LM7805, U2 LM7812

Commit message: Poprawiony tranzystor
Parts:
- moved Q1 5.00 mm to (114.8, 147.2), turned to 180 degrees
Connections:
- Q1 pad 1: Net-(Q1-Pad1) -> GND
- Q1 pad 2: Net-(D1-Pad1) -> Net-(Q1-Pad2)
- Q1 pad 3: GND -> Net-(D1-Pad1)
- R6 pad 1: Net-(Q1-Pad1) -> Net-(Q1-Pad2)
Routing:
- net Net-(Q1-Pad2): track 0.00 -> 7.32 mm
- net Net-(Q1-Pad1): track 5.35 -> 0.00 mm
- net Net-(D1-Pad1): track 19.4 -> 17.5 mm
Changed lines of the file:
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@@
     (links 63)
     (no_connects 4)
-    (area 20.275 21.155 268.033334 184.675)
+    (area 24.275 19.655 264.783334 180.175)
     (thickness 1.6)
     (drawings 0)
-    (tracks 117)
+    (tracks 118)
     (zones 0)
     (modules 32)
@@
   )
   (setup
-    (last_trace_width 1.5)
+    (last_trace_width 0.25)
     (user_trace_width 0.5)
     (user_trace_width 0.75)
@@
       (outputformat 4)
       (mirror false)
-      (drillshape 0)
+      (drillshape 1)
       (scaleselection 1)
       (outputdirectory ""))
@@
   (net 16 "Net-(J1-Pad2)")
   (net 17 "Net-(J1-Pad4)")
-  (net 18 "Net-(Q1-Pad1)")
-  (net 19 "Net-(R1-Pad1)")
-  (net 20 "Net-(R2-Pad2)")
-  (net 21 "Net-(R3-Pad1)")
-  (net 22 "Net-(R4-Pad2)")
-  (net 23 "Net-(R5-Pad1)")
-  (net 24 "Net-(J3-Pad1)")
+  (net 18 "Net-(R1-Pad1)")
+  (net 19 "Net-(R2-Pad2)")
+  (net 20 "Net-(R3-Pad1)")
+  (net 21 "Net-(R4-Pad2)")
+  (net 22 "Net-(R5-Pad1)")
+  (net 23 "Net-(J3-Pad1)")
+  (net 24 "Net-(Q1-Pad2)")
   (net_class Default "To jest domyślna klasa połączeń."
     (clearance 0.2)
@@
     (add_net "Net-(J1-Pad4)")
     (add_net "Net-(J3-Pad1)")
-    (add_net "Net-(Q1-Pad1)")
+    (add_net "Net-(Q1-Pad2)")
     (add_net "Net-(R1-Pad1)")
     (add_net "Net-(R2-Pad2)")
@@
   )
   (module TO_SOT_Packages_THT:TO-92_Inline_Narrow_Oval (layer F.Cu)
-    (at 111.75 143.25 270)
+    (at 114.75 147.25 180)
     (descr "TO-92 leads in-line, narrow, oval pads, drill 0.6mm (see NXP sot054_po.pdf)")
     (tags "to-92 sc-43 sc-43a sot54 PA33 transistor")
-    (fp_text reference Q1 (at 0 -4 270) (layer F.SilkS)
-      (effects (font (size 1 1) (thickness 0.15)))
-    )
-    (fp_text value Q_NPN_BCE (at 0 3 270) (layer F.Fab)
+    (fp_text reference Q1 (at 0 -4 180) (layer F.SilkS)
+      (effects (font (size 1 1) (thickness 0.15)))
+    )
+    (fp_text value Q_NPN_BCE (at 0 3 180) (layer F.Fab)
       (effects (font (size 1 1) (thickness 0.15)))
     )
@@
     (fp_line (start -1.4 -2.65) (end 3.95 -2.65) (layer F.CrtYd) (width 0.05))
     (fp_line (start 3.95 1.95) (end 3.95 -2.65) (layer F.CrtYd) (width 0.05))
-    (pad 2 thru_hole oval (at 1.27 0 90) (size 0.89916 1.50114) (drill 0.6) (layers *.Cu *.Mask F.SilkS)
+    (pad 2 thru_hole oval (at 1.27 0) (size 0.89916 1.50114) (drill 0.6) (layers *.Cu *.Mask F.SilkS)
+      (net 24 "Net-(Q1-Pad2)"))
+    (pad 3 thru_hole oval (at 2.54 0) (size 0.89916 1.50114) (drill 0.6) (layers *.Cu *.Mask F.SilkS)
       (net 6 "Net-(D1-Pad1)"))
-    (pad 3 thru_hole oval (at 2.54 0 90) (size 0.89916 1.50114) (drill 0.6) (layers *.Cu *.Mask F.SilkS)
-      (net 2 GND))
-    (pad 1 thru_hole oval (at 0 0 90) (size 0.89916 1.50114) (drill 0.6) (layers *.Cu *.Mask F.SilkS)
-      (net 18 "Net-(Q1-Pad1)"))
+    (pad 1 thru_hole oval (at 0 0) (size 0.89916 1.50114) (drill 0.6) (layers *.Cu *.Mask F.SilkS)
+      (net 2 GND))
     (model TO_SOT_Packages_THT.3dshapes/TO-92_Inline_Narrow_Oval.wrl
       (at (xyz 0.05 0 0))
@@
     (fp_line (start 3.80876 5.08) (end 3.80876 -5.08) (layer F.SilkS) (width 0.15))
     (pad 1 thru_hole circle (at 0 0 90) (size 2.30124 2.30124) (drill 1.00076) (layers *.Cu *.SilkS *.Mask)
-      (net 19 "Net-(R1-Pad1)"))
+      (net 18 "Net-(R1-Pad1)"))
     (pad 2 thru_hole circle (at 30 0 90) (size 2.30124 2.30124) (drill 1.19888) (layers *.Cu *.SilkS *.Mask)
       (net 17 "Net-(J1-Pad4)"))
@@
     (fp_line (start 3.80876 5.08) (end 3.80876 -5.08) (layer F.SilkS) (width 0.15))
     (pad 1 thru_hole circle (at 0 0 90) (size 2.30124 2.30124) (drill 1.00076) (layers *.Cu *.SilkS *.Mask)
-      (net 19 "Net-(R1-Pad1)"))
+      (net 18 "Net-(R1-Pad1)"))
     (pad 2 thru_hole circle (at 30 0 90) (size 2.30124 2.30124) (drill 1.19888) (layers *.Cu *.SilkS *.Mask)
-      (net 20 "Net-(R2-Pad2)"))
+      (net 19 "Net-(R2-Pad2)"))
   )
   (module Resistors_ThroughHole:Resistor_Horizontal_RM30mm (layer F.Cu)
@@
     (fp_line (start 3.80876 5.08) (end 3.80876 -5.08) (layer F.SilkS) (width 0.15))
     (pad 1 thru_hole circle (at 0 0 90) (size 2.30124 2.30124) (drill 1.00076) (layers *.Cu *.SilkS *.Mask)
-      (net 21 "Net-(R3-Pad1)"))
+      (net 20 "Net-(R3-Pad1)"))
     (pad 2 thru_hole circle (at 30 0 90) (size 2.30124 2.30124) (drill 1.19888) (layers *.Cu *.SilkS *.Mask)
-      (net 20 "Net-(R2-Pad2)"))
+      (net 19 "Net-(R2-Pad2)"))
   )
   (module Resistors_ThroughHole:Resistor_Horizontal_RM30mm (layer F.Cu)
@@
     (fp_line (start 3.80876 5.08) (end 3.80876 -5.08) (layer F.SilkS) (width 0.15))
     (pad 1 thru_hole circle (at 0 0 90) (size 2.30124 2.30124) (drill 1.00076) (layers *.Cu *.SilkS *.Mask)
-      (net 21 "Net-(R3-Pad1)"))
+      (net 20 "Net-(R3-Pad1)"))
     (pad 2 thru_hole circle (at 30 0 90) (size 2.30124 2.30124) (drill 1.19888) (layers *.Cu *.SilkS *.Mask)
-      (net 22 "Net-(R4-Pad2)"))
+      (net 21 "Net-(R4-Pad2)"))
   )
   (module Resistors_ThroughHole:Resistor_Horizontal_RM30mm (layer F.Cu)
@@
     (fp_line (start 3.80876 5.08) (end 3.80876 -5.08) (layer F.SilkS) (width 0.15))
     (pad 1 thru_hole circle (at 0 0 90) (size 2.30124 2.30124) (drill 1.00076) (layers *.Cu *.SilkS *.Mask)
-      (net 23 "Net-(R5-Pad1)"))
+      (net 22 "Net-(R5-Pad1)"))
     (pad 2 thru_hole circle (at 30 0 90) (size 2.30124 2.30124) (drill 1.19888) (layers *.Cu *.SilkS *.Mask)
-      (net 22 "Net-(R4-Pad2)"))
+      (net 21 "Net-(R4-Pad2)"))
   )
   (module Resistors_ThroughHole:Resistor_Horizontal_RM7mm (layer F.Cu)
@@
     (fp_line (start 1.27 1.27) (end 1.27 -1.27) (layer F.SilkS) (width 0.15))
     (pad 1 thru_hole circle (at 0 0 90) (size 1.99898 1.99898) (drill 1.00076) (layers *.Cu *.SilkS *.Mask)
-      (net 18 "Net-(Q1-Pad1)"))
+      (net 24 "Net-(Q1-Pad2)"))
     (pad 2 thru_hole circle (at 7.62 0 90) (size 1.99898 1.99898) (drill 1.00076) (layers *.Cu *.SilkS *.Mask)
-      (net 24 "Net-(J3-Pad1)"))
+      (net 23 "Net-(J3-Pad1)"))
   )
   (module Resistors_ThroughHole:Resistor_Horizontal_RM7mm (layer F.Cu)
@@
       (net 17 "Net-(J1-Pad4)"))
     (pad 12 thru_hole circle (at 14.2 -6 270) (size 3 3) (drill 1.3) (layers *.Cu *.Mask)
-      (net 23 "Net-(R5-Pad1)"))
+      (net 22 "Net-(R5-Pad1)"))
     (pad 2 thru_hole circle (at 1.95 -5.95 270) (size 2.5 2.5) (drill 1) (layers *.Cu *.Mask F.SilkS)
       (net 6 "Net-(D1-Pad1)"))
@@
     (fp_line (start -1.27 1.27) (end 1.27 1.27) (layer F.SilkS) (width 0.15))
     (pad 1 thru_hole rect (at 0 0) (size 2.2352 2.2352) (drill 1.016) (layers *.Cu *.Mask F.SilkS)
-      (net 24 "Net-(J3-Pad1)"))
+      (net 23 "Net-(J3-Pad1)"))
     (model Pin_Headers.3dshapes/Pin_Header_Straight_1x01.wrl
       (at (xyz 0 0 0))
@@
   (segment (start 96.25 114.25) (end 96.25 113.5) (width 1.5) (layer F.Cu) (net 5))
   (segment (start 96.25 113.5) (end 96.25 109.5) (width 1.5) (layer F.Cu) (net 5))
+  (segment (start 112.21 147.25) (end 107.91306 147.25) (width 1) (layer F.Cu) (net 6))
+  (segment (start 107.91306 147.25) (end 107.75254 147.41052) (width 1) (layer F.Cu) (net 6))
   (segment (start 103.5 150.5) (end 98.1 150.5) (width 1) (layer F.Cu) (net 6))
   (segment (start 98.1 150.5) (end 97.55 149.95) (width 1) (layer F.Cu) (net 6))
@@
   (segment (start 107.75254 149.49746) (end 107.75254 147.41052) (width 1) (layer F.Cu) (net 6))
   (segment (start 106.75 150.5) (end 107.75254 149.49746) (width 1) (layer F.Cu) (net 6))
-  (segment (start 107.75254 147.41052) (end 107.75254 145.24746) (width 1) (layer F.Cu) (net 6))
-  (segment (start 108.48 144.52) (end 111.75 144.52) (width 1) (layer F.Cu) (net 6))
-  (segment (start 107.75254 145.24746) (end 108.48 144.52) (width 1) (layer F.Cu) (net 6))
   (segment (start 103.5 147.96) (end 103.5 145.87) (width 1) (layer F.Cu) (net 7))
   (segment (start 103.5 145.87) (end 102.75 145.12) (width 1) (layer F.Cu) (net 7))
@@
   (segment (start 31.7 113.45) (end 33.25 113.45) (width 3) (layer F.Cu) (net 17))
   (segment (start 29.7 115.45) (end 31.7 113.45) (width 3) (layer F.Cu) (net 17))
-  (segment (start 111.75 143.25) (end 116.75 143.25) (width 1) (layer F.Cu) (net 18))
-  (segment (start 116.75 143.25) (end 117 143.5) (width 1) (layer F.Cu) (net 18))
-  (segment (start 29.7 151.3) (end 41 151.3) (width 3) (layer F.Cu) (net 19))
-  (segment (start 41 121.3) (end 52.25 121.3) (width 3) (layer F.Cu) (net 20))
-  (segment (start 52.25 151.3) (end 63.7 151.3) (width 3) (layer F.Cu) (net 21))
-  (segment (start 63.7 151.3) (end 63.75 151.25) (width 3) (layer F.Cu) (net 21))
-  (segment (start 63.75 121.25) (end 75 121.25) (width 3) (layer F.Cu) (net 22))
-  (segment (start 75 151.25) (end 84.05 151.25) (width 3) (layer F.Cu) (net 23))
-  (segment (start 84.05 151.25) (end 85.3 150) (width 3) (layer F.Cu) (net 23))
-  (segment (start 112.25 136.5) (end 116.38 136.5) (width 1.5) (layer F.Cu) (net 24))
-  (segment (start 116.38 136.5) (end 117 135.88) (width 1.5) (layer F.Cu) (net 24))
+  (segment (start 29.7 151.3) (end 41 151.3) (width 3) (layer F.Cu) (net 18))
+  (segment (start 41 121.3) (end 52.25 121.3) (width 3) (layer F.Cu) (net 19))
+  (segment (start 52.25 151.3) (end 63.7 151.3) (width 3) (layer F.Cu) (net 20))
+  (segment (start 63.7 151.3) (end 63.75 151.25) (width 3) (layer F.Cu) (net 20))
+  (segment (start 63.75 121.25) (end 75 121.25) (width 3) (layer F.Cu) (net 21))
+  (segment (start 75 151.25) (end 84.05 151.25) (width 3) (layer F.Cu) (net 22))
+  (segment (start 84.05 151.25) (end 85.3 150) (width 3) (layer F.Cu) (net 22))
+  (segment (start 112.25 136.5) (end 116.38 136.5) (width 1.5) (layer F.Cu) (net 23))
+  (segment (start 116.38 136.5) (end 117 135.88) (width 1.5) (layer F.Cu) (net 23))
+  (segment (start 113.48 147.25) (end 113.48 144.02) (width 1) (layer F.Cu) (net 24))
+  (segment (start 114 143.5) (end 117 143.5) (width 1) (layer F.Cu) (net 24))
+  (segment (start 113.48 144.02) (end 114 143.5) (width 1) (layer F.Cu) (net 24))
+  (segment (start 116.75 143.25) (end 117 143.5) (width 1) (layer F.Cu) (net 24))
   (zone (net 2) (net_name GND) (layer F.Cu) (hatch edge 0.508)
     (connect_pads (clearance 0.508))
